File: KiCad/Lab8-Schematic.kicad_sch (KiCad schematic)
At the start: 37 parts, among them J1 Command Generator, J2 Line Sensor, M1 Motor, M2 Motor, Q2 LTR3208E, SW1 Reset, SW2 SW-SPDT, U1 PIC32MX170F256B, U2 L293NE, U3 MCP6294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

Commit message: Changed back to RB11 for SDI, seeing data in pulseview, D2 uneven and matching oscilloscope
Connections:
- net at U1.24 (RB13): no longer J1.6 (Pin_6)
- net at U1.26 (RB15): now also J1.6 (Pin_6)
Changed lines of the file:
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@@
   (junction (at 88.9 43.18) (diameter 0) (color 0 0 0 0)
   )
+  (wire (pts (xy 101.6 52.07) (xy 101.6 76.2))
+    (stroke (width 0) (type default))
+  )
   (wire (pts (xy 201.93 81.28) (xy 201.93 85.09))
     (stroke (width 0) (type default))
@@
     (stroke (width 0) (type default))
   )
-  (wire (pts (xy 88.9 85.09) (xy 95.25 85.09))
-    (stroke (width 0) (type default))
-  )
   (wire (pts (xy 17.78 193.04) (xy 53.34 193.04))
     (stroke (width 0) (type default))
@@
     (stroke (width 0) (type default))
   )
-  (wire (pts (xy 106.68 113.03) (xy 90.17 113.03))
-    (stroke (width 0) (type default))
-  )
   (wire (pts (xy 55.88 157.48) (xy 55.88 160.02))
     (stroke (width 0) (type default))
@@
     (stroke (width 0) (type default))
   )
+  (wire (pts (xy 88.9 80.01) (xy 97.79 80.01))
+    (stroke (width 0) (type default))
+  )
   (wire (pts (xy 55.88 157.48) (xy 67.31 157.48))
     (stroke (width 0) (type default))
@@
     (stroke (width 0) (type default))
   )
-  (wire (pts (xy 106.68 80.01) (xy 106.68 113.03))
-    (stroke (width 0) (type default))
-  )
   (wire (pts (xy 88.9 167.64) (xy 88.9 179.07))
     (stroke (width 0) (type default))
@@
     (stroke (width 0) (type default))
   )
+  (wire (pts (xy 95.25 90.17) (xy 95.25 116.84))
+    (stroke (width 0) (type default))
+  )
   (wire (pts (xy 146.05 58.42) (xy 154.94 58.42))
     (stroke (width 0) (type default))
@@
     (stroke (width 0) (type default))
   )
-  (wire (pts (xy 101.6 76.2) (xy 101.6 52.07))
+  (wire (pts (xy 97.79 80.01) (xy 97.79 105.41))
     (stroke (width 0) (type default))
   )
@@
     (stroke (width 0) (type default))
   )
-  (wire (pts (xy 90.17 113.03) (xy 90.17 116.84))
+  (wire (pts (xy 90.17 105.41) (xy 90.17 116.84))
     (stroke (width 0) (type default))
   )
@@
     (stroke (width 0) (type default))
   )
+  (wire (pts (xy 88.9 90.17) (xy 95.25 90.17))
+    (stroke (width 0) (type default))
+  )
   (wire (pts (xy 97.79 171.45) (xy 105.41 171.45))
     (stroke (width 0) (type default))
@@
     (stroke (width 0) (type default))
   )
+  (wire (pts (xy 97.79 105.41) (xy 90.17 105.41))
+    (stroke (width 0) (type default))
+  )
   (wire (pts (xy 170.18 97.79) (xy 170.18 88.9))
     (stroke (width 0) (type default))
@@
     (stroke (width 0) (type default))
   )
-  (wire (pts (xy 95.25 85.09) (xy 95.25 116.84))
-    (stroke (width 0) (type default))
-  )
   (wire (pts (xy 161.29 63.5) (xy 134.62 63.5))
     (stroke (width 0) (type default))
@@
     (stroke (width 0) (type default))
   )
-  (wire (pts (xy 88.9 80.01) (xy 106.68 80.01))
-    (stroke (width 0) (type default))
-  )

Commit message: IR circuit debugged in hardware, awaiting softare testing, schematic updated to reflect hardware changes
Parts:
- renumbered 10k2 to 10k, 10k1 to 15k
Connections:
- net +3.3V: no longer 15k.1
- net +5V: now also 0.1uF2.1, 15k.1, U5.4 (V+)
- net at 10k.1, 15k.2, R9.2: now also U5.3 (+); no longer U5.2 (-)
- net at R7.2, U3.1: now also U5.2 (-); no longer U5.3 (+)

Commit message: debugging beacon service
Connections:
- net at U1.17 (5VT/RB8): now also J1.4 (Pin_4)
- net at U1.22 (RB11): no longer J1.4 (Pin_4)

Commit message: Post check off kicad save
Parts:
- removed R7: 100k, symbol ME218_BaseLib:Res1
- R6: value 68k -> 470k
Connections:
- net V(out): now also U1.21 (PGEC2/5VT/RB10); no longer U1.2 (RA0)
- net at U3.1, U5.2 (-): now also R6.2
- net LED: now reaches U1.11 (RB4)
Other:
- moved on the sheet: R6
